File: xiphos.kicad_pcb (KiCad board)
At the start: 2 copper layers, 292.4 x 97.5 mm, 76 parts

Commit message: Adjust magsafe position
Parts:
- moved MAG1 5.83 mm to (137.5, 130.8)
- moved MAG2 5.83 mm to (282.4, 130.8)
