File: xiphos.kicad_sch (KiCad schematic)
At the start: 42 parts

Commit message: cleanup
Parts:
- MCU1, MCU2: symbol huntercooh:nice_nano_raw21 -> huntercook:nice_nano_raw21
- S1, S10, S11, S12, S13, S14, S15, S16, S17, S19, S2, S20, S21, S22, S23, S24, S25, S26, S27, S28, S29, S3, S30, S31, S32, S33, S34, S35, S4, S5, S6, S7, S8, S9: symbol huntercooh:PG1316S -> huntercook:PG1316S
Changed lines of the file:
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@@
 	)
 (symbol
-		(lib_id "huntercooh:PG1316S")
+		(lib_id "huntercook:PG1316S")
 		(at 55.88 71.12 0)
 		(unit 1)
@@
 	)
 (symbol
-		(lib_id "huntercooh:PG1316S")
+		(lib_id "huntercook:PG1316S")
 		(at 38.1 97.79 0)
 		(unit 1)
@@
 	)
 (symbol
-		(lib_id "huntercooh:PG1316S")
+		(lib_id "huntercook:PG1316S")
 		(at 72.39 97.79 0)
 		(unit 1)
@@
 	)
 (symbol
-		(lib_id "huntercooh:nice_nano_raw21")
+		(lib_id "huntercook:nice_nano_raw21")
 		(at 204.47 71.12 0)
 		(mirror y)
@@
 	)
 (symbol
-		(lib_id "huntercooh:PG1316S")
+		(lib_id "huntercook:PG1316S")
 		(at 88.9 44.45 0)
 		(unit 1)
@@
 	)
 (symbol
-		(lib_id "huntercooh:PG1316S")
+		(lib_id "huntercook:PG1316S")
 		(at 72.39 71.12 0)
 		(unit 1)
@@
 	)
 (symbol
-		(lib_id "huntercooh:PG1316S")
+		(lib_id "huntercook:PG1316S")
 		(at 38.1 44.45 0)
 		(unit 1)
@@
 	)
 (symbol
-		(lib_id "huntercooh:PG1316S")
+		(lib_id "huntercook:PG1316S")
 		(at 105.41 125.73 0)
 		(unit 1)
@@
 	)
 (symbol
-		(lib_id "huntercooh:PG1316S")
+		(lib_id "huntercook:PG1316S")
 		(at 88.9 125.73 0)
 		(unit 1)
@@
 	)
 (symbol
-		(lib_id "huntercooh:PG1316S")
+		(lib_id "huntercook:PG1316S")
 		(at 55.88 97.79 0)
 		(unit 1)
@@
 	)
 (symbol
-		(lib_id "huntercooh:PG1316S")
+		(lib_id "huntercook:PG1316S")
 		(at 88.9 97.79 0)
 		(unit 1)
@@
 	)
 (symbol
-		(lib_id "huntercooh:PG1316S")
+		(lib_id "huntercook:PG1316S")
 		(at 88.9 71.12 0)
 		(unit 1)
@@
 	)
 (symbol
-		(lib_id "huntercooh:PG1316S")
+		(lib_id "huntercook:PG1316S")
 		(at 38.1 71.12 0)
 		(unit 1)
@@
 	)
 (symbol
-		(lib_id "huntercooh:PG1316S")
+		(lib_id "huntercook:PG1316S")
 		(at 105.41 97.79 0)
 		(unit 1)
@@
 	)
 (symbol
-		(lib_id "huntercooh:PG1316S")
+		(lib_id "huntercook:PG1316S")
 		(at 72.39 44.45 0)
 		(unit 1)
@@
 	)
 (symbol
-		(lib_id "huntercooh:PG1316S")
+		(lib_id "huntercook:PG1316S")
 		(at 55.88 44.45 0)
 		(unit 1)
@@
 	)
 (symbol
-		(lib_id "huntercooh:PG1316S")
+		(lib_id "huntercook:PG1316S")
 		(at 105.41 44.45 0)
 		(unit 1)
@@
 	)
 (symbol
-		(lib_id "huntercooh:PG1316S")
+		(lib_id "huntercook:PG1316S")
 		(at 105.41 71.12 0)
 		(unit 1)
@@
 	)
 (symbol
-		(lib_id "huntercooh:PG1316S")
+		(lib_id "huntercook:PG1316S")
 		(at 309.75 71.12 0)
 		(unit 1)
@@
 	)
 (symbol
-		(lib_id "huntercooh:PG1316S")
+		(lib_id "huntercook:PG1316S")
 		(at 291.97 97.79 0)
 		(unit 1)
@@
 	)
 (symbol
-		(lib_id "huntercooh:PG1316S")
+		(lib_id "huntercook:PG1316S")
 		(at 326.26 97.79 0)
 		(unit 1)
@@
 	)
 (symbol
-		(lib_id "huntercooh:nice_nano_raw21")
+		(lib_id "huntercook:nice_nano_raw21")
 		(at 458.34 71.12 0)
 		(mirror y)
@@
 	)
 (symbol
-		(lib_id "huntercooh:PG1316S")
+		(lib_id "huntercook:PG1316S")
 		(at 342.77 44.45 0)
 		(unit 1)
@@
 	)
 (symbol
-		(lib_id "huntercooh:PG1316S")
+		(lib_id "huntercook:PG1316S")
 		(at 326.26 71.12 0)
 		(unit 1)
@@
 	)
 (symbol
-		(lib_id "huntercooh:PG1316S")
+		(lib_id "huntercook:PG1316S")
 		(at 291.97 44.45 0)
 		(unit 1)
@@
 	)
 (symbol
-		(lib_id "huntercooh:PG1316S")
+		(lib_id "huntercook:PG1316S")
 		(at 359.28 125.73 0)
 		(unit 1)
@@
 	)
 (symbol
-		(lib_id "huntercooh:PG1316S")
+		(lib_id "huntercook:PG1316S")
 		(at 342.77 125.73 0)
 		(unit 1)
@@
 	)
 (symbol
-		(lib_id "huntercooh:PG1316S")
+		(lib_id "huntercook:PG1316S")
 		(at 309.75 97.79 0)
 		(unit 1)
@@
 	)
 (symbol
-		(lib_id "huntercooh:PG1316S")
+		(lib_id "huntercook:PG1316S")
 		(at 342.77 97.79 0)
 		(unit 1)
@@
 	)
 (symbol
-		(lib_id "huntercooh:PG1316S")
+		(lib_id "huntercook:PG1316S")
 		(at 342.77 71.12 0)
 		(unit 1)
@@
 	)
 (symbol
-		(lib_id "huntercooh:PG1316S")
+		(lib_id "huntercook:PG1316S")
 		(at 291.97 71.12 0)
 		(unit 1)
@@
 	)
 (symbol
-		(lib_id "huntercooh:PG1316S")
+		(lib_id "huntercook:PG1316S")
 		(at 359.28 97.79 0)
 		(unit 1)
@@
 	)
 (symbol
-		(lib_id "huntercooh:PG1316S")
+		(lib_id "huntercook:PG1316S")
 		(at 326.26 44.45 0)
 		(unit 1)
@@
 	)
 (symbol
-		(lib_id "huntercooh:PG1316S")
+		(lib_id "huntercook:PG1316S")
 		(at 309.75 44.45 0)
 		(unit 1)
@@
 	)
 (symbol
-		(lib_id "huntercooh:PG1316S")
+		(lib_id "huntercook:PG1316S")
 		(at 359.28 44.45 0)
 		(unit 1)
@@
 	)
 (symbol
-		(lib_id "huntercooh:PG1316S")
+		(lib_id "huntercook:PG1316S")
 		(at 359.28 71.12 0)
 		(unit 1)

Commit message: Adjust magsafe position
Parts:
- CONN1, CONN2: LCSC (none) -> C505023
- MCU1, MCU2: footprint ceoloide:mcu_nice_nano -> PCM_marbastlib-xp-promicroish:nice_nano_AH_USBup; LCSC (none) -> DNP; now not fitted
- PWR1, PWR2: LCSC (none) -> C2911519
- RST1, RST2: LCSC (none) -> C79174
- S1, S10, S11, S12, S13, S14, S15, S16, S17, S19, S2, S20, S21, S22, S23, S24, S25, S26, S27, S28, S29, S3, S30, S31, S32, S33, S34, S35, S4, S5, S6, S7, S8, S9: LCSC (none) -> C9900170245
Other:
- moved on the sheet: CONN2, PWR2, RST2, S19, S20, S21, S22, S23, S24, S25, S26, S27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
